File: midi_keyboard/midi_keyboard.kicad_pcb (KiCad board)
At the start: 2 copper layers, 152.9 x 146.1 mm, 16 parts, among them J1 Conn_01x12, SW1 RotaryEncoder_Switch_MP, SW2 SW_Push, SW3 SW_Push, SW4 SW_Push, U1 CD74HC4067M, U3 ER_OLEDM0.91_1x-I2C

Commit message: file upload edits
Parts:
- RV1, RV2: footprint Potentiometer_THT:Potentiometer_Bourns_PTA1543_Single_Slide -> Potentiometer_THT:Potentiometer_Bourns_PTA3043_Single_Slide
- moved BZ2 47.4 mm to (166.6, 162.2)
- moved BZ3 47.4 mm to (147.5, 175.8)
- moved U1 47.4 mm to (136.6, 121.3)
- moved D3 47.4 mm to (25.0, 131.9)
- moved J1 47.4 mm to (36.9, 135.8)
- moved RV1 47.4 mm to (104.7, 122.8)
- moved RV2 47.4 mm to (91.8, 122.6)
- moved SW1 47.4 mm to (26.2, 118.8)
- moved SW2 47.4 mm to (78.3, 97.2)
- moved SW3 47.4 mm to (57.1, 97.0)
- moved A1 47.4 mm to (130.5, 108.4)
- moved BZ1 47.4 mm to (148.3, 147.1)
- moved D1 47.4 mm to (96.7, 129.6)
- moved SW4 47.4 mm to (35.2, 97.3)
- moved D2 47.4 mm to (159.5, 131.9)
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Routing:
- net GND: track 391.9 -> 470.3 mm
- net /SCL: track 136.8 -> 144.8 mm
- net /SDA: track 135.3 -> 143.3 mm
- net +5V: track 123.1 -> 131.1 mm
Other:
- board size 152.9 x 146.1 mm -> 152.9 x 164.9 mm
