File: midi_keyboard/midi_keyboard.kicad_sch (KiCad schematic)
At the start: 16 parts, among them J1 Conn_01x12, SW1 RotaryEncoder_Switch_MP, SW2 SW_Push, SW3 SW_Push, SW4 SW_Push, U1 CD74HC4067M, U3 ER_OLEDM0.91_1x-I2C

Commit message: file upload edits
Parts:
- RV1, RV2: footprint Potentiometer_THT:Potentiometer_Bourns_PTA1543_Single_Slide -> Potentiometer_THT:Potentiometer_Bourns_PTA3043_Single_Slide
Changed lines of the file:
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@@
 			)
 		)
-		(property "Footprint" "Potentiometer_THT:Potentiometer_Bourns_PTA1543_Single_Slide"
+		(property "Footprint" "Potentiometer_THT:Potentiometer_Bourns_PTA3043_Single_Slide"
 			(at 86.36 25.4 0)
 			(hide yes)
@@
 			)
 		)
-		(property "Footprint" "Potentiometer_THT:Potentiometer_Bourns_PTA1543_Single_Slide"
+		(property "Footprint" "Potentiometer_THT:Potentiometer_Bourns_PTA3043_Single_Slide"
 			(at 86.36 48.26 0)
 			(hide yes)
